File: Schematics/System Diagrams/Full System Diagram rev1.sch (EAGLE design)
At the start: 12 parts, among them K1 RELAY

Commit message: added current sensor into the system diagram and added some schematic pictures
Parts:
- removed F1: (no value), HyTechSymbols:FUSE
- added FUSE1: (no value), HyTechSymbols:FUSE
Other:
- moved on the sheet: K1
