File: Schematics/Cell Charger BMS/Cell Charger BMS rev1.brd (EAGLE design)
At the start: 114.6 x 175.6 mm, 120 parts, among them J1_B 0R, J2_B 0R, J3_B 0R, J4_B 0R, J5_B 0R, J6_B 0R, J7_B 0R, J8_B 0R, Q2 NSV1C201MZ4, U2 LTC6811-2

Commit message: charger BMS WiP
Parts:
- removed CELL0, CELL1, CELL2, CELL3, CELL4, CELL5, CELL6, CELL7, CELL8, CELL9: BATTERY_SPRING_SPRING_CONTACT, HyTechDevices:CONTACT_SPRING
- removed ISOSPI_B: ISOSPI, HyTechDevices:NANO-FIT_VERTICAL-2
- removed RM_B: 100R, HyTechDevices:0603-RES
- added X1: CONNECTOR-10NANO-FIT_VERTICAL-10, HyTechDevices:1053101210
- added X2: CONNECTOR-2NANO-FIT_VERTICAL-2, HyTechDevices:1053091202
- moved U$13 10.2 mm to (-8.97, 4.05)
- moved U$27 8.78 mm to (5.00, 149.0)
- moved U$14 6.75 mm to (109.3, 5.41)
Connections:
- removed net CC9: CELL9.P$1, F9.P$1
- removed net GPIO1_B: U2.27
- removed net GPIO2_B: U2.28
- removed net GPIO3_B: U2.29
- removed net GPIO4_B: U2.32
- removed net GPIO5_B: U2.33
- new net N$3: F9.P$1, X1.P$10
- net CC0: now also X1.P$1; no longer CELL0.P$1
- net CC1: now also X1.P$2; no longer CELL1.P$1
- net CC2: now also X1.P$3; no longer CELL2.P$1
- net CC3: now also X1.P$4; no longer CELL3.P$1
- net CC4: now also X1.P$5; no longer CELL4.P$1
- net CC5: now also X1.P$6; no longer CELL5.P$1
- net CC6: now also X1.P$7; no longer CELL6.P$1
- net CC7: now also X1.P$8; no longer CELL7.P$1
- net CC8: now also X1.P$9; no longer CELL8.P$1
- net ISOSPI-M: now also X2.2; no longer ISOSPI_B.P$2, RM_B.2
- net ISOSPI-P: now also X2.1; no longer ISOSPI_B.P$1, RM_B.1
Routing:
- net CC8: track 22.3 -> 152.9 mm, vias 1 -> 2
- net CC7: track 21.1 -> 117.1 mm, vias 1 -> 2
- net N$3: track 0.00 -> 93.7 mm
- net CC6: track 22.9 -> 101.8 mm, vias 1 -> 2
- net CC0: track 24.2 -> 87.7 mm
- net CC5: track 21.7 -> 84.4 mm, vias 1 -> 2
- net CC1: track 14.1 -> 69.2 mm
- net CC2: track 23.3 -> 77.0 mm
- net VREF2_B: track 8.47 -> 61.1 mm, vias 1 -> 2
- net CC4: track 24.5 -> 74.8 mm
- net V-_A: track 94.6 -> 144.4 mm
- net CC3: track 22.6 -> 67.9 mm
- net ISOSPI-P: track 42.2 -> 7.11 mm
- net CC9: track 23.6 -> 0.00 mm, vias 1 -> 0
- net V-_B: track 513.2 -> 536.3 mm, vias 18 -> 20
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Other:
- board size 114.6 x 175.6 mm -> 134.9 x 165.1 mm
- board text added: "+"
- board text added: "10"
- board text added: "11"
- board text added: "12"
- board text added: "9"
- board text added: "DANGER HIGH VOLTAGE"
- board text added: "DRIVE_A"

Commit message: charger BMS almost done
Parts:
- moved DRAIN6:PFET 18.3 mm to (88.1, 90.0)
- moved J1_B 18.3 mm to (121.4, 104.8)
- moved J2_B 18.3 mm to (119.5, 104.8)
- moved J3_B 18.3 mm to (117.6, 104.8)
- moved J4_B 18.3 mm to (115.7, 104.8)
- moved RB1_B 18.3 mm to (119.8, 82.0)
- moved C1_B 18.3 mm to (119.8, 72.5)
- moved C2_B 18.3 mm to (119.8, 75.7)
- moved C3_B 18.3 mm to (106.7, 121.9)
- moved C4_B 18.3 mm to (102.7, 126.3)
- moved C8_B 18.3 mm to (116.8, 58.2)
- moved DRAIN2:C 18.3 mm to (86.6, 41.1)
- moved DRAIN2:LED1 18.3 mm to (88.1, 32.4)
- moved DRAIN2:PFET 18.3 mm to (88.1, 36.7)
- moved DRAIN2:R 18.3 mm to (91.7, 41.1)
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Routing:
- net V-_B: track 536.3 -> 552.4 mm
- net V-_A: track 144.4 -> 146.9 mm
Other:
- board size 134.9 x 165.1 mm -> 124.5 x 149.9 mm
- board text added: "HyTech Racing 2021 Cell Charger BMS rev 1 Designed by Leo Pozdneev, based on BMS Segment rev 14 by Arvind Srinivasan"
- board text removed: "#"
- board text removed: "+"
- board text removed: "10"
- board text removed: "11"
- board text removed: "12"
- board text removed: "9"
- board text removed: "DRIVE_A"
- board text removed: "HyTech Racing 2020 BMS Segment rev14 Designed by Arvind Srinivasan, based on rev10 by Yvonne Yeh"
