File: Schematics/Cell Charger BMS/Cell Charger BMS rev1.sch (EAGLE design)
At the start: 43 parts, among them J1_B 0R, J2_B 0R, J3_B 0R, J4_B 0R, J5_B 0R, J6_B 0R, J7_B 0R, J8_B 0R, Q2 NSV1C201MZ4, U2 LTC6811-2, X1 CONNECTOR-10NANO-FIT_VERTICAL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, X2 CONNECTOR-2NANO-FIT_VERTICAL-2

Commit message: charger BMS almost done
Changed lines of the file:
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@@
 <attribute name="FRAME_DESCRIPTION" value="Upper LTC6811 IC"/>
-</part>
-<part name="U$23" library="HyTechFrames" deviceset="FRAME_B" device="">
-<attribute name="ENGINEER" value="Arvind Srinivasan"/>
-<attribute name="FRAME_DESCRIPTION" value="Lower LTC6811 IC and Cell Thermistor Test Connection"/>
-</part>
-<part name="U$24" library="HyTechFrames" deviceset="FRAME_B" device="">
-<attribute name="ENGINEER" value="Arvind Srinivasan"/>
-<attribute name="FRAME_DESCRIPTION" value="Upper 9 Cell Connections and Cell Voltage Test Connection"/>
 </part>
 <part name="U$25" library="HyTechFrames" deviceset="FRAME_B" device="">
@@
 </parts>
 <sheets>
-<sheet>
-<description>Upper 9 Cell Connections and Cell Voltage Test Connection</description>
-<plain>
-</plain>
-<instances>
-<instance part="U$24" gate="G$1" x="-431.8" y="0" smashed="yes"/>
-<instance part="U$24" gate="G$2" x="-168.91" y="0" smashed="yes">
-<attribute name="LAST_DATE_TIME" x="-92.71" y="2.54" size="2.54" layer="94"/>
-<attribute name="DRAWING_NAME" x="-73.66" y="22.86" size="2.54" layer="94"/>
-<attribute name="SHEET" x="-20.32" y="2.54" size="2.54" layer="94"/>
-<attribute name="FRAME_DESCRIPTION" x="-102.87" y="10.16" size="2.54" layer="94"/>
-<attribute name="ENGINEER" x="-149.86" y="22.86" size="2.54" layer="94"/>
-</instance>
-</instances>
-<busses>
-</busses>
-<nets>
-</nets>
-</sheet>
 <sheet>
 <description>Lower 9 Cell Connections</description>
@@
 </nets>
 </sheet>
-<sheet>
-<description>Lower LTC6811 IC and Cell Thermistor Test Connection</description>
-<plain>
-</plain>
-<instances>
-<instance part="U$23" gate="G$1" x="-431.8" y="0" smashed="yes"/>
-<instance part="U$23" gate="G$2" x="-168.91" y="0" smashed="yes">
-<attribute name="LAST_DATE_TIME" x="-92.71" y="2.54" size="2.54" layer="94"/>
-<attribute name="DRAWING_NAME" x="-73.66" y="22.86" size="2.54" layer="94"/>
-<attribute name="SHEET" x="-20.32" y="2.54" size="2.54" layer="94"/>
-<attribute name="FRAME_DESCRIPTION" x="-102.87" y="10.16" size="2.54" layer="94"/>
-<attribute name="ENGINEER" x="-149.86" y="22.86" size="2.54" layer="94"/>
-</instance>
-</instances>
-<busses>
-</busses>
-<nets>
-</nets>
-</sheet>
